File: hardware/theta-remote-release.kicad_pcb (KiCad board)
At the start: 2 copper layers, 48 x 39 mm, 21 parts, among them P1 Li-Po Battery, SW1 POWER, SW2 PUSH-SW, U1 AE-FT234X, U2 MCP73831, U3 ESP-WROOM-02, U4 TPS63000

Commit message: add reference
Changed lines of the file:
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@@
-(kicad_pcb (version 4) (host pcbnew "(2015-10-11 BZR 6260)-product")
+(kicad_pcb (version 4) (host pcbnew 4.0.1-stable)
   (general
     (links 46)
     (no_connects 0)
-    (area 109.7 64.8 216.728573 143.200001)
+    (area 97.300001 64.8 216.728573 143.200001)
     (thickness 1.6)
-    (drawings 42)
+    (drawings 50)
     (tracks 153)
     (zones 0)
@@
     (pad_to_mask_clearance 0.2)
     (aux_axis_origin 0 0)
-    (visible_elements FFFFEFFF)
+    (visible_elements FFFFFFFF)
     (pcbplotparams
       (layerselection 0x010f0_80000001)
@@
       (net 16 +BATT))
   )
+  (gr_line (start 122.3 121) (end 122.3 90) (angle 90) (layer F.Fab) (width 0.2))
+  (gr_line (start 201.5 124.2) (end 125.5 124.2) (angle 90) (layer F.Fab) (width 0.2))
+  (gr_line (start 204.7 90) (end 204.7 121) (angle 90) (layer F.Fab) (width 0.2))
+  (gr_line (start 125.5 86.8) (end 201.5 86.8) (angle 90) (layer F.Fab) (width 0.2))
+  (gr_arc (start 125.5 121) (end 125.5 124.2) (angle 90) (layer F.Fab) (width 0.2))
+  (gr_arc (start 125.5 90) (end 122.3 90) (angle 90) (layer F.Fab) (width 0.2))
+  (gr_arc (start 201.5 90) (end 201.5 86.8) (angle 90) (layer F.Fab) (width 0.2))
+  (gr_arc (start 201.5 121) (end 204.7 121) (angle 90) (layer F.Fab) (width 0.2))
   (dimension 16.5 (width 0.1) (layer F.Fab)
     (gr_text 16.5mm (at 126.75 78.15) (layer F.Fab)
@@
   (segment (start 157 101) (end 157 103) (width 0.25) (layer F.Cu) (net 9))
   (segment (start 156.725 100.725) (end 157 101) (width 0.25) (layer F.Cu) (net 9))
-  (segment (start 158.5 99.275) (end 159.275 99.275) (width 0.25) (layer F.Cu) (net 10))
-  (segment (start 154 119.5) (end 154 121) (width 0.25) (layer F.Cu) (net 10))
-  (segment (start 153.5 119) (end 154 119.5) (width 0.25) (layer F.Cu) (net 10))
-  (segment (start 152.5 119) (end 153.5 119) (width 0.25) (layer F.Cu) (net 10))
-  (segment (start 152 118.5) (end 152.5 119) (width 0.25) (layer F.Cu) (net 10))
-  (segment (start 152 105.5) (end 152 118.5) (width 0.25) (layer F.Cu) (net 10))
-  (segment (start 152.5 105) (end 152 105.5) (width 0.25) (layer F.Cu) (net 10))
-  (segment (start 159.5 105) (end 152.5 105) (width 0.25) (layer F.Cu) (net 10))
-  (segment (start 160 104.5) (end 159.5 105) (width 0.25) (layer F.Cu) (net 10))
-  (segment (start 160 100) (end 160 104.5) (width 0.25) (layer F.Cu) (net 10))
-  (segment (start 159.275 99.275) (end 160 100) (width 0.25) (layer F.Cu) (net 10))
+  (segment (start 154 121) (end 154 119.4) (width 0.25) (layer F.Cu) (net 10) (status 400000))
+  (segment (start 159.275 99.275) (end 158.5 99.275) (width 0.25) (layer F.Cu) (net 10) (status 800000))
+  (segment (start 159.7 99.7) (end 159.275 99.275) (width 0.25) (layer F.Cu) (net 10))
+  (segment (start 159.7 104.2) (end 159.7 99.7) (width 0.25) (layer F.Cu) (net 10))
+  (segment (start 159.1 104.8) (end 159.7 104.2) (width 0.25) (layer F.Cu) (net 10))
+  (segment (start 152.4 104.8) (end 159.1 104.8) (width 0.25) (layer F.Cu) (net 10))
+  (segment (start 152 105.2) (end 152.4 104.8) (width 0.25) (layer F.Cu) (net 10))
+  (segment (start 152 118.5) (end 152 105.2) (width 0.25) (layer F.Cu) (net 10))
+  (segment (start 152.5 119) (end 152 118.5) (width 0.25) (layer F.Cu) (net 10))
+  (segment (start 153.6 119) (end 152.5 119) (width 0.25) (layer F.Cu) (net 10))
+  (segment (start 154 119.4) (end 153.6 119) (width 0.25) (layer F.Cu) (net 10))
   (segment (start 158.5 99.275) (end 158.775 99.275) (width 0.25) (layer F.Cu) (net 10))
   (segment (start 149.5 100.725) (end 149.5 103) (width 0.25) (layer F.Cu) (net 11))
@@
       )
     )
+  )
+  (zone (net 0) (net_name "") (layer F.Cu) (hatch edge 0.508)
+    (connect_pads (clearance 0.508))
+    (min_thickness 0.254)
+    (keepout (tracks not_allowed) (vias not_allowed) (copperpour not_allowed))
+    (fill (arc_segments 16) (thermal_gap 0.508) (thermal_bridge_width 0.508))
+    (polygon
+      (pts
+        (xy 165.8 120.8) (xy 160 120.8) (xy 160 103.2) (xy 165.8 103.2) (xy 165.8 120.8)
+      )
+    )
+  )
+  (zone (net 0) (net_name "") (layer B.Cu) (hatch edge 0.508)
+    (connect_pads (clearance 0.508))
+    (min_thickness 0.254)
+    (keepout (tracks not_allowed) (vias not_allowed) (copperpour not_allowed))
+    (fill (arc_segments 16) (thermal_gap 0.508) (thermal_bridge_width 0.508))
+    (polygon
+      (pts
+        (xy 165.8 120.8) (xy 160 120.8) (xy 160 103.2) (xy 165.8 103.2) (xy 165.8 120.8)
+      )
+    )

Commit message: add 1.0.0
Parts:
- removed D3: STATUS, theta-remote-release:LED
- removed U4: TPS63000, theta-remote-release:TPS63000
- added C3: 4.7uF, theta-remote-release:SMD2012, B.Cu at (135.4, 81.0)
- added CN1: ZX62R-B-5P, theta-remote-release:ZX62R-B-5P, F.Cu at (138.5, 70.5)
- added CN2: DEBUG, theta-remote-release:Debug, F.Cu at (150.5, 90.0)
- C1, C2: value 4.7μF -> 4.7uF; moved to B.Cu
- D1: value CHARGE -> CHG; footprint theta-remote-release:LED -> theta-remote-release:SMD2012_LED
- D2: value POWER -> STAT; footprint theta-remote-release:LED -> theta-remote-release:SMD2012_LED
- P1: value Li-Po Battery -> Li-Po 3.7V; footprint theta-remote-release:PH-2P-TOP-SIDE -> theta-remote-release:Li-Po
- R1: value 2kΩ -> 10k; moved to B.Cu
- R2, R3, R4, R5: value 10kΩ -> 10k
- R6: value 4.7kΩ -> 10k
- R7: value 470Ω -> 100; moved to B.Cu
- R8: value 470Ω -> 10k
- R9: value 470Ω -> 100
- SW1: footprint theta-remote-release:SS12D01G4 -> theta-remote-release:ESP2020
- SW2: value PUSH-SW -> SHUTTER; footprint theta-remote-release:PUSH-SW -> theta-remote-release:TVAF17-WEC-R
- U1: value AE-FT234X -> MCP73831; footprint theta-remote-release:AE-FT234X -> TO_SOT_Packages_SMD:SOT-23-5; moved to B.Cu
- U2: value MCP73831 -> ESP-WROOM-02; footprint TO_SOT_Packages_SMD:SOT-23-5 -> theta-remote-release:esp-wroom-02; moved to B.Cu
- U3: value ESP-WROOM-02 -> MCP1825S-3002E/DB; footprint theta-remote-release:esp-wroom-02 -> TO_SOT_Packages_SMD:SOT-223; moved to B.Cu
- moved R7 43.7 mm to (143.7, 78.5), turned to 180 degrees
- moved U3 35.7 mm to (129.6, 79.8)
- moved R9 34.6 mm to (143.5, 86.5), turned to 0 degrees
- moved U1 28.3 mm to (143.7, 81.0), turned to 180 degrees
- moved R3 27.7 mm to (133.5, 88.0), turned to 180 degrees
- moved R8 27.7 mm to (143.5, 92.5), turned to 0 degrees
- moved D1 24.2 mm to (138.5, 93.0), turned to 180 degrees
- moved SW2 22.6 mm to (138.5, 83.0), turned to 180 degrees
- moved R1 22.3 mm to (140.6, 81.0), turned to 90 degrees
- moved C2 20.5 mm to (146.9, 81.0), turned to 90 degrees
- moved R5 20.4 mm to (133.5, 89.5), turned to 180 degrees
- moved SW1 17.8 mm to (150.0, 82.0), turned to 270 degrees
- moved R6 17.1 mm to (133.5, 91.0), turned to 180 degrees
- moved D2 17.0 mm to (138.5, 98.0), turned to 180 degrees
- moved R4 16.3 mm to (133.5, 97.0), turned to 180 degrees
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Connections:
- D2 pad 2: +3V3 -> +3V
- R2 pad 1: +3V3 -> +3V
- R2 pad 2: Net-(R2-Pad2) -> Net-(CN2-Pad1)
- R3 pad 1: +3V3 -> +3V
- R3 pad 2: Net-(R3-Pad2) -> Net-(CN2-Pad2)
- R4 pad 1: +3V3 -> +3V
- R5 pad 1: Net-(R5-Pad1) -> +3V
- R5 pad 2: GND -> Net-(R5-Pad2)
- R6 pad 1: +3V3 -> GND
- R6 pad 2: /IO0 -> Net-(R6-Pad2)
- R7 pad 2: /STAT -> /CHG
- R8 pad 1: Net-(D2-Pad1) -> +3V
- R8 pad 2: GND -> /IO5
- R9 pad 1: Net-(D3-Pad1) -> Net-(D2-Pad1)
- SW1 pad 2: Net-(C2-Pad1) -> Net-(SW1-Pad2)
- SW1 pad 3: +BATT -> Net-(C2-Pad1)
- SW2 pad 1: /IO0 -> /IO5
- U1 pad 1: +5V -> /CHG
- U1 pad 3: Net-(U1-Pad3) -> Net-(C2-Pad1)
- U1 pad 4: Net-(U1-Pad4) -> +5V
- U2 pad 1: /STAT -> +3V
- U2 pad 2: GND -> Net-(R4-Pad2)
- U2 pad 3: Net-(C2-Pad1) -> (no net)
- U2 pad 4: +5V -> (no net)
- U2 pad 5: Net-(R1-Pad2) -> (no net)
- U3 pad 1: +3V3 -> Net-(SW1-Pad2)
- U3 pad 2: Net-(R2-Pad2) -> GND
- U3 pad 3: (no net) -> +3V
- U3 pad 4: (no net) -> GND
Routing:
- net +3V3: track 60.5 -> 0.00 mm, vias 4 -> 0
- net +3V: track 0.00 -> 42.4 mm, vias 0 -> 2
- net Net-(U1-Pad4): track 36.4 -> 0.00 mm
- net Net-(U1-Pad3): track 34.8 -> 0.00 mm
- net Net-(R3-Pad2): track 31.5 -> 0.00 mm
- net Net-(CN2-Pad2): track 0.00 -> 25.3 mm, vias 0 -> 2
- net /STAT: track 23.4 -> 0.00 mm, vias 2 -> 0
- net Net-(D1-Pad1): track 2.51 -> 23.1 mm, vias 0 -> 1
- net Net-(SW1-Pad2): track 0.00 -> 20.2 mm
- net Net-(C2-Pad1): track 38.0 -> 20.3 mm
- net /IO5: track 0.00 -> 15.6 mm, vias 0 -> 1
- net Net-(CN2-Pad1): track 0.00 -> 15.0 mm, vias 0 -> 1
- net +BATT: track 13.4 -> 0.00 mm
- net /IO4: track 16.7 -> 3.28 mm, vias 0 -> 1
- net Net-(D2-Pad1): track 2.51 -> 14.2 mm, vias 0 -> 2
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Other:
- board size 48 x 39 mm -> 29 x 36 mm
